Commit message: add another plugin for singlehandmode, the original plugin is used for leftandright configurtion, for cob, we should use the single hand version

File: robotiq_s_model_visualization/cfg/robotiq_hand_macro.urdf.xacro (robot description, xacro)
@@ -6,5 +6,6 @@
 there are multiple hands then a prefix followed by an "_" is needed.
 -->
-<robot xmlns:xacro="http://www.ros.org/wiki/xacro" name="robotiq_hand">
+<!--<robot xmlns:xacro="http://www.ros.org/wiki/xacro" name="robotiq_hand">-->
+<robot xmlns:xacro="http://www.ros.org/wiki/xacro">
   <xacro:macro name="robotiq_finger" params="prefix">
     <!-- Link list -->
@@ -632,11 +633,12 @@
     </gazebo>
   </xacro:macro>
-  <xacro:macro name="robotiq_hand" params="prefix *origin reflect parent">
+  <!--<xacro:macro name="robotiq_hand" params="prefix *origin reflect parent">-->
+  <xacro:macro name="robotiq_hand" params="prefix reflect">
     <!-- joint attaching parent link to robotiq hand -->
-    <joint name="${prefix}robotiq_hand_joint" type="fixed">
-      <insert_block name="origin"/>
-      <parent link="${parent}"/>
-      <child link="${prefix}palm"/>
-    </joint>
+    <!--<joint name="${prefix}robotiq_hand_joint" type="fixed">-->
+      <!--<insert_block name="origin"/>-->
+      <!--<parent link="${parent}"/>-->
+      <!--<child link="${prefix}palm"/>-->
+    <!--</joint>-->
     <!-- Insert the fingers -->
     <xacro:robotiq_finger prefix="${prefix}finger_1_"/>

Commit message: add dae instead of stl, since dae includes color and material information

File: robotiq_s_model_visualization/cfg/robotiq_hand_macro.urdf.xacro (robot description, xacro)
@@ -15,5 +15,5 @@
         <origin xyz="0 0 0" rpy="0 0 0"/>
         <geometry>
-          <mesh filename="package://robotiq_s_model_visualization/meshes/s-model_articulated/visual/link_0.STL" />
+          <mesh filename="package://robotiq_s_model_visualization/meshes/s-model_articulated/visual/link_0.dae" />
         </geometry>
         <material name="green">
@@ -24,5 +24,5 @@
         <origin rpy="0 0 0" xyz="0 0 0"/>
         <geometry>
-          <mesh filename="package://robotiq_s_model_visualization/meshes/s-model_articulated/collision/link_0.STL" />
+          <mesh filename="package://robotiq_s_model_visualization/meshes/s-model_articulated/collision/link_0.dae" />
         </geometry>
         <material name="yellow">
@@ -45,5 +45,5 @@
         <origin rpy="0 0 ${3.1416/2}" xyz="0 0.05717 0"/>
         <geometry>
-          <mesh filename="package://robotiq_s_model_visualization/meshes/s-model_articulated/visual/link_1.STL" />
+          <mesh filename="package://robotiq_s_model_visualization/meshes/s-model_articulated/visual/link_1.dae" />
         </geometry>
         <material name="green"/>
@@ -52,5 +52,5 @@
         <origin rpy="0 0 ${3.1416/2}" xyz="0 0.05717 0"/>
         <geometry>
-          <mesh filename="package://robotiq_s_model_visualization/meshes/s-model_articulated/collision/link_1.STL"/>
+          <mesh filename="package://robotiq_s_model_visualization/meshes/s-model_articulated/collision/link_1.dae"/>
         </geometry>
         <material name="yellow">
@@ -78,5 +78,5 @@
         <origin rpy="0 0 ${3.1416/2}" xyz="0 0.03810 0.0075"/>
         <geometry>
-          <mesh filename="package://robotiq_s_model_visualization/meshes/s-model_articulated/visual/link_2.STL" />
+          <mesh filename="package://robotiq_s_model_visualization/meshes/s-model_articulated/visual/link_2.dae" />
         </geometry>
         <material name="green"/>
@@ -85,5 +85,5 @@
         <origin rpy="0 0 ${3.1416/2}" xyz="0 0.03810 0.0075"/>
           <geometry>
-            <mesh filename="package://robotiq_s_model_visualization/meshes/s-model_articulated/collision/link_2.STL"/>
+            <mesh filename="package://robotiq_s_model_visualization/meshes/s-model_articulated/collision/link_2.dae"/>
           </geometry>
         <material name="yellow"/>
@@ -109,5 +109,5 @@
         <origin xyz="0 0 0" rpy="0 0 0"/>
         <geometry>
-          <mesh filename="package://robotiq_s_model_visualization/meshes/s-model_articulated/visual/link_3.STL" />
+          <mesh filename="package://robotiq_s_model_visualization/meshes/s-model_articulated/visual/link_3.dae" />
         </geometry>
         <material name="green"/>
@@ -116,5 +116,5 @@
         <origin xyz="0 0 0" rpy="0 0 0"/>
         <geometry>
-          <mesh filename="package://robotiq_s_model_visualization/meshes/s-model_articulated/collision/link_3.STL"/>
+          <mesh filename="package://robotiq_s_model_visualization/meshes/s-model_articulated/collision/link_3.dae"/>
         </geometry>
         <material name="yellow"/>
@@ -650,5 +650,5 @@
         <visual>
           <geometry>
-            <mesh filename="package://robotiq_s_model_visualization/meshes/s-model_articulated/visual/palm.STL" />
+            <mesh filename="package://robotiq_s_model_visualization/meshes/s-model_articulated/visual/palm.dae" />
           </geometry>
           <material name="green">

File: robotiq_s_model_visualization/cfg/robotiq_hand_macro_with_gazebo_plugin.urdf.xacro (robot description, xacro)
@@ -19,5 +19,5 @@
         <origin xyz="0 0 0" rpy="0 0 0"/>
         <geometry>
-          <mesh filename="package://robotiq_s_model_visualization/meshes/s-model_articulated/visual/link_0.STL" />
+          <mesh filename="package://robotiq_s_model_visualization/meshes/s-model_articulated/visual/link_0.dae" />
         </geometry>
         <material name="green">
@@ -28,5 +28,5 @@
         <origin rpy="0 0 0" xyz="0 0 0"/>
         <geometry>
-          <mesh filename="package://robotiq_s_model_visualization/meshes/s-model_articulated/collision/link_0.STL" />
+          <mesh filename="package://robotiq_s_model_visualization/meshes/s-model_articulated/collision/link_0.dae" />
         </geometry>
         <material name="yellow">
@@ -49,5 +49,5 @@
         <origin rpy="0 0 ${3.1416/2}" xyz="0 0.05717 0"/>
         <geometry>
-          <mesh filename="package://robotiq_s_model_visualization/meshes/s-model_articulated/visual/link_1.STL" />
+          <mesh filename="package://robotiq_s_model_visualization/meshes/s-model_articulated/visual/link_1.dae" />
         </geometry>
         <material name="green"/>
@@ -56,5 +56,5 @@
         <origin rpy="0 0 ${3.1416/2}" xyz="0 0.05717 0"/>
         <geometry>
-          <mesh filename="package://robotiq_s_model_visualization/meshes/s-model_articulated/collision/link_1.STL"/>
+          <mesh filename="package://robotiq_s_model_visualization/meshes/s-model_articulated/collision/link_1.dae"/>
         </geometry>
         <material name="yellow">
@@ -82,5 +82,5 @@
         <origin rpy="0 0 ${3.1416/2}" xyz="0 0.03810 0.0075"/>
         <geometry>
-          <mesh filename="package://robotiq_s_model_visualization/meshes/s-model_articulated/visual/link_2.STL" />
+          <mesh filename="package://robotiq_s_model_visualization/meshes/s-model_articulated/visual/link_2.dae" />
         </geometry>
         <material name="green"/>
@@ -89,5 +89,5 @@
         <origin rpy="0 0 ${3.1416/2}" xyz="0 0.03810 0.0075"/>
           <geometry>
-            <mesh filename="package://robotiq_s_model_visualization/meshes/s-model_articulated/collision/link_2.STL"/>
+            <mesh filename="package://robotiq_s_model_visualization/meshes/s-model_articulated/collision/link_2.dae"/>
           </geometry>
         <material name="yellow"/>
@@ -113,5 +113,5 @@
         <origin xyz="0 0 0" rpy="0 0 0"/>
         <geometry>
-          <mesh filename="package://robotiq_s_model_visualization/meshes/s-model_articulated/visual/link_3.STL" />
+          <mesh filename="package://robotiq_s_model_visualization/meshes/s-model_articulated/visual/link_3.dae" />
         </geometry>
         <material name="green"/>
@@ -120,5 +120,5 @@
         <origin xyz="0 0 0" rpy="0 0 0"/>
         <geometry>
-          <mesh filename="package://robotiq_s_model_visualization/meshes/s-model_articulated/collision/link_3.STL"/>
+          <mesh filename="package://robotiq_s_model_visualization/meshes/s-model_articulated/collision/link_3.dae"/>
         </geometry>
         <material name="yellow"/>
@@ -653,5 +653,5 @@
         <visual>
           <geometry>
-            <mesh filename="package://robotiq_s_model_visualization/meshes/s-model_articulated/visual/palm.STL" />
+            <mesh filename="package://robotiq_s_model_visualization/meshes/s-model_articulated/visual/palm.dae" />
           </geometry>
           <material name="green">

File: robotiq_s_model_visualization/cfg/s-model_articulated_macro.xacro (robot description, xacro)
@@ -16,5 +16,5 @@
 			<visual>
 				<geometry>
-					<mesh filename="package://robotiq_s_model_visualization/meshes/s-model_articulated/visual/palm.STL" />
+					<mesh filename="package://robotiq_s_model_visualization/meshes/s-model_articulated/visual/palm.dae" />
 				</geometry>
 				<material name="gray">
@@ -24,5 +24,5 @@
 			<collision>
 				<geometry>
-					<mesh filename="package://robotiq_s_model_visualization/meshes/s-model_articulated/collision/palm.STL" />
+					<mesh filename="package://robotiq_s_model_visualization/meshes/s-model_articulated/collision/palm.dae" />
 				</geometry>
 				<material name="yellow">

File: robotiq_s_model_visualization/cfg/s-model_finger_articulated_macro.xacro (robot description, xacro)
@@ -12,5 +12,5 @@
 				<origin xyz="0.020 0 0" rpy="0 0 0"/>
 				<geometry>
-					<mesh filename="package://robotiq_s_model_visualization/meshes/s-model_articulated/visual/link_0.STL" />
+					<mesh filename="package://robotiq_s_model_visualization/meshes/s-model_articulated/visual/link_0.dae" />
 				</geometry>
 				<material name="gray">
@@ -21,5 +21,5 @@
 				<origin xyz="0.020 0 0" rpy="0 0 0"/>
 				<geometry>
-					<mesh filename="package://robotiq_s_model_visualization/meshes/s-model_articulated/collision/link_0.STL" />
+					<mesh filename="package://robotiq_s_model_visualization/meshes/s-model_articulated/collision/link_0.dae" />
 				</geometry>
 				<material name="yellow">
@@ -37,5 +37,5 @@
 				<origin xyz="0.050 -.028 0" rpy="0 0 -0.52"/>
 				<geometry>
-					<mesh filename="package://robotiq_s_model_visualization/meshes/s-model_articulated/visual/link_1.STL" />
+					<mesh filename="package://robotiq_s_model_visualization/meshes/s-model_articulated/visual/link_1.dae" />
 				</geometry>
 				<material name="gray"/>
@@ -44,5 +44,5 @@
 				<origin xyz="0.050 -.028 0" rpy="0 0 -0.52"/>
 				<geometry>
-					<mesh filename="package://robotiq_s_model_visualization/meshes/s-model_articulated/collision/link_1.STL" />
+					<mesh filename="package://robotiq_s_model_visualization/meshes/s-model_articulated/collision/link_1.dae" />
 				</geometry>
 				<material name="yellow"/>
@@ -63,5 +63,5 @@
 				<origin xyz="0.039 0 0.0075" rpy="0 0 0"/>
 				<geometry>
-					<mesh filename="package://robotiq_s_model_visualization/meshes/s-model_articulated/visual/link_2.STL" />
+					<mesh filename="package://robotiq_s_model_visualization/meshes/s-model_articulated/visual/link_2.dae" />
 				</geometry>
 				<material name="gray"/>
@@ -70,5 +70,5 @@
 				<origin xyz="0.039 0 0.0075" rpy="0 0 0"/>
 				<geometry>
-					<mesh filename="package://robotiq_s_model_visualization/meshes/s-model_articulated/collision/link_2.STL" />
+					<mesh filename="package://robotiq_s_model_visualization/meshes/s-model_articulated/collision/link_2.dae" />
 				</geometry>
 				<material name="yellow"/>
@@ -84,5 +84,5 @@
 				<origin xyz="0 0 0" rpy="0 0 0.52"/>
 				<geometry>
-					<mesh filename="package://robotiq_s_model_visualization/meshes/s-model_articulated/visual/link_3.STL" />
+					<mesh filename="package://robotiq_s_model_visualization/meshes/s-model_articulated/visual/link_3.dae" />
 				</geometry>
 				<material name="gray"/>
@@ -91,5 +91,5 @@
 				<origin xyz="0 0 0" rpy="0 0 0.52"/>
 				<geometry>
-					<mesh filename="package://robotiq_s_model_visualization/meshes/s-model_articulated/collision/link_3.STL" />
+					<mesh filename="package://robotiq_s_model_visualization/meshes/s-model_articulated/collision/link_3.dae" />
 				</geometry>
 				<material name="yellow"/>

File: robotiq_s_model_visualization/cfg/s-model_mesh_macro.xacro (robot description, xacro)
@@ -5,5 +5,5 @@
 			<visual>
 				<geometry>
-					<mesh filename="package://robotiq_s_model_visualization/meshes/s-model/visual/GRIPPER_OPEN_PALM.stl" />
+					<mesh filename="package://robotiq_s_model_visualization/meshes/s-model/visual/GRIPPER_OPEN_PALM.dae" />
 				</geometry>
 				<material name="green">
@@ -13,5 +13,5 @@
 			<collision>
 				<geometry>
-					<mesh filename="package://robotiq_s_model_visualization/meshes/s-model/collision/GRIPPER_OPEN_PALM.stl" />
+					<mesh filename="package://robotiq_s_model_visualization/meshes/s-model/collision/GRIPPER_OPEN_PALM.dae" />
 				</geometry>
 				<material name="yellow">
@@ -23,5 +23,5 @@
 			<visual>
 				<geometry>
-					<mesh filename="package://robotiq_s_model_visualization/meshes/s-model/visual/GRIPPER_OPEN_FINGER_1.stl" />
+					<mesh filename="package://robotiq_s_model_visualization/meshes/s-model/visual/GRIPPER_OPEN_FINGER_1.dae" />
 				</geometry>
 				<material name="green"/>
@@ -29,5 +29,5 @@
 			<collision>
 				<geometry>
-					<mesh filename="package://robotiq_s_model_visualization/meshes/s-model/collision/GRIPPER_OPEN_FINGER_1.stl" />
+					<mesh filename="package://robotiq_s_model_visualization/meshes/s-model/collision/GRIPPER_OPEN_FINGER_1.dae" />
 				</geometry>
 				<material name="yellow"/>
@@ -37,5 +37,5 @@
 			<visual>
 				<geometry>
-					<mesh filename="package://robotiq_s_model_visualization/meshes/s-model/visual/GRIPPER_OPEN_FINGER_2.stl" />
+					<mesh filename="package://robotiq_s_model_visualization/meshes/s-model/visual/GRIPPER_OPEN_FINGER_2.dae" />
 				</geometry>
 				<material name="green"/>
@@ -43,5 +43,5 @@
 			<collision>
 				<geometry>
-					<mesh filename="package://robotiq_s_model_visualization/meshes/s-model/collision/GRIPPER_OPEN_FINGER_2.stl" />
+					<mesh filename="package://robotiq_s_model_visualization/meshes/s-model/collision/GRIPPER_OPEN_FINGER_2.dae" />
 				</geometry>
 				<material name="yellow"/>
@@ -51,5 +51,5 @@
 			<visual>
 				<geometry>
-					<mesh filename="package://robotiq_s_model_visualization/meshes/s-model/visual/GRIPPER_OPEN_FINGER_3.stl" />
+					<mesh filename="package://robotiq_s_model_visualization/meshes/s-model/visual/GRIPPER_OPEN_FINGER_3.dae" />
 				</geometry>
 				<material name="green"/>
@@ -57,5 +57,5 @@
 			<collision>
 				<geometry>
-					<mesh filename="package://robotiq_s_model_visualization/meshes/s-model/collision/GRIPPER_OPEN_FINGER_3.stl" />
+					<mesh filename="package://robotiq_s_model_visualization/meshes/s-model/collision/GRIPPER_OPEN_FINGER_3.dae" />
 				</geometry>
 				<material name="yellow"/>
