Commit message: compose all robot together

File: robotiq_s_model_visualization/cfg/common.gazebo.xacro (robot description, xacro)
@@ -1,14 +1,15 @@
 <?xml version="1.0"?>
 <robot xmlns:xacro="http://ros.org/wiki/xacro" >
-  <xacro:arg name="namespace_without_slash" default="left_hand"/>
-  <!-- <gazebo>
-    <plugin name="RobotiqHandPlugin" filename="libRobotiqHandPlugin.so">
-      <side>$(arg namespace_without_slash)</side>
-    </plugin>
-  </gazebo> -->
-  <gazebo>
-    <plugin name="RobotiqHandPluginControlMsg" filename="libRobotiqHandPlugin_controlMsg.so">
-      <side>$(arg namespace_without_slash)</side>
-    </plugin>
-  </gazebo>
+  <xacro:macro name="robotiq_common_gazebo" params="namespace_without_slash">
+    <!-- <gazebo>
+      <plugin name="RobotiqHandPlugin" filename="libRobotiqHandPlugin.so">
+        <side>${namespace_without_slash}</side>
+      </plugin>
+    </gazebo> -->
+    <gazebo>
+      <plugin name="RobotiqHandPluginControlMsg" filename="libRobotiqHandPlugin_controlMsg.so">
+        <side>${namespace_without_slash}</side>
+      </plugin>
+    </gazebo>
+  </xacro:macro>
 </robot>

File: robotiq_s_model_visualization/cfg/robotiq_hand_robot.urdf.xacro (robot description, xacro)
@@ -7,7 +7,6 @@
   <!-- common stuff -->
   <!-- https://answers.ros.org/question/216975/loading-variables-with-xacroinclude/ -->
-  <xacro:include filename="$(find robotiq_s_model_visualization)/cfg/common.gazebo.xacro">
-    <xacro:arg name="namespace_without_slash" value="$(arg namespace_without_slash)"/>
-  </xacro:include>
+  <xacro:include filename="$(find robotiq_s_model_visualization)/cfg/common.gazebo.xacro" />
+  <xacro:robotiq_common_gazebo namespace_without_slash="$(arg namespace_without_slash)" />
   <!-- robotiq_hand -->
   <xacro:include filename="$(find robotiq_s_model_visualization)/cfg/robotiq_hand_macro.urdf.xacro" />
