Commit message: restructure gazebo plugin and use cob_plugin isntead of the vanilla gazebo plugin. because it can target on specific joint names

File: robotiq_s_model_visualization/cfg/robotiq_hand.plugin.gazebo.xacro (robot description, xacro)
@@ -1,5 +1,5 @@
 <?xml version="1.0"?>
 <robot xmlns:xacro="http://ros.org/wiki/xacro" >
-  <xacro:macro name="robotiq_common_gazebo" params="namespace_without_slash">
+  <xacro:macro name="robotiq_hand_plugin_gazebo" params="namespace_without_slash">
     <!-- <gazebo>
       <plugin name="RobotiqHandPlugin" filename="libRobotiqHandPlugin.so">

File: robotiq_s_model_visualization/cfg/robotiq_hand_robot.urdf.xacro (robot description, xacro)
@@ -5,12 +5,9 @@
   <xacro:arg name="prefix_without_underscore" default="left_hand"/>
   <xacro:arg name="prefix" default="$(arg prefix_without_underscore)_"/>
-  <!-- common stuff -->
   <!-- https://answers.ros.org/question/216975/loading-variables-with-xacroinclude/ -->
-  <xacro:include filename="$(find robotiq_s_model_visualization)/cfg/common.gazebo.xacro" />
-  <xacro:robotiq_common_gazebo namespace_without_slash="$(arg namespace_without_slash)" />
-  <!-- robotiq_hand -->
+  <xacro:include filename="$(find robotiq_s_model_visualization)/cfg/robotiq_hand.plugin.gazebo.xacro" />
+  <xacro:robotiq_hand_plugin_gazebo namespace_without_slash="$(arg namespace_without_slash)" />
   <xacro:include filename="$(find robotiq_s_model_visualization)/cfg/robotiq_hand_macro.urdf.xacro" />
   <link name="world"/>
-  <!-- robotiq_hand -->
   <xacro:robotiq_hand prefix="$(arg prefix)" parent="world" reflect="-1">
     <origin rpy="0 0 0" xyz="0 0 1.0"/>
